File: PCBdesign/kicad/Synapse/Current Mirror_1.kicad_sch (KiCad schematic)
At the start: 5 parts, among them IC2 ALD1105PBL

Commit message: Annotate schematics (auto via kicad) and generate netlists.
Parts:
- renumbered RC1* to RC1*1, RI1* to RI1*1
Changed lines of the file:
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@@
 		(in_pos_files yes)
 		(dnp no)
-		(property "Reference" "#PWR?"
+		(property "Reference" "#PWR014"
 			(at 160.02 104.5972 0)
 			(hide yes)
@@
 			(project "Synapse_LPS"
 				(path "/af4a7426-c915-4fd8-a9a0-d1d0653890c7/efb34e1f-b4a1-4d0a-a367-85b7a624cd54"
-					(reference "#PWR?")
+					(reference "#PWR014")
 					(unit 1)
 				)
@@
 		(in_pos_files yes)
 		(dnp no)
-		(property "Reference" "RI1*"
+		(property "Reference" "RI1*1"
 			(at 166.37 102.0572 0)
 			(show_name no)
@@
 			(project "Synapse_LPS"
 				(path "/af4a7426-c915-4fd8-a9a0-d1d0653890c7/efb34e1f-b4a1-4d0a-a367-85b7a624cd54"
-					(reference "RI1*")
+					(reference "RI1*1")
 					(unit 1)
 				)
@@
 		(in_pos_files yes)
 		(dnp no)
-		(property "Reference" "#PWR?"
+		(property "Reference" "#PWR012"
 			(at 96.52 131.2672 0)
 			(hide yes)
@@
 			(project "Synapse_LPS"
 				(path "/af4a7426-c915-4fd8-a9a0-d1d0653890c7/efb34e1f-b4a1-4d0a-a367-85b7a624cd54"
-					(reference "#PWR?")
+					(reference "#PWR012")
 					(unit 1)
 				)
@@
 		(in_pos_files yes)
 		(dnp no)
-		(property "Reference" "#PWR?"
+		(property "Reference" "#PWR013"
 			(at 118.11 131.2672 0)
 			(hide yes)
@@
 			(project "Synapse_LPS"
 				(path "/af4a7426-c915-4fd8-a9a0-d1d0653890c7/efb34e1f-b4a1-4d0a-a367-85b7a624cd54"
-					(reference "#PWR?")
+					(reference "#PWR013")
 					(unit 1)
 				)
@@
 		(in_pos_files yes)
 		(dnp no)
-		(property "Reference" "RC1*"
+		(property "Reference" "RC1*1"
 			(at 103.886 95.9612 90)
 			(show_name no)
@@
 			(project "Synapse_LPS"
 				(path "/af4a7426-c915-4fd8-a9a0-d1d0653890c7/efb34e1f-b4a1-4d0a-a367-85b7a624cd54"
-					(reference "RC1*")
+					(reference "RC1*1")
 					(unit 1)
 				)
@@
 		(in_pos_files yes)
 		(dnp no)
-		(property "Reference" "#PWR?"
+		(property "Reference" "#PWR011"
 			(at 83.82 131.2672 0)
 			(hide yes)
@@
 			(project "Synapse_LPS"
 				(path "/af4a7426-c915-4fd8-a9a0-d1d0653890c7/efb34e1f-b4a1-4d0a-a367-85b7a624cd54"
-					(reference "#PWR?")
+					(reference "#PWR011")
 					(unit 1)
 				)
