File: PCBdesign/kicad/Synapse/Current Mirror_2.kicad_sch (KiCad schematic)
At the start: 5 parts, among them IC3 ALD1105PBL

Commit message: Annotate schematics (auto via kicad) and generate netlists.
Parts:
- renumbered RC2* to RC2*1, RI2* to RI2*1
Changed lines of the file:
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@@
 		(in_pos_files yes)
 		(dnp no)
-		(property "Reference" "RI2*"
+		(property "Reference" "RI2*1"
 			(at 161.036 96.7232 0)
 			(show_name no)
@@
 			(project "Synapse_LPS"
 				(path "/af4a7426-c915-4fd8-a9a0-d1d0653890c7/c9470723-b410-4315-971f-b3c2471482a7"
-					(reference "RI2*")
+					(reference "RI2*1")
 					(unit 1)
 				)
@@
 		(in_pos_files yes)
 		(dnp no)
-		(property "Reference" "#PWR?"
+		(property "Reference" "#PWR018"
 			(at 154.94 99.5172 0)
 			(hide yes)
@@
 			(project "Synapse_LPS"
 				(path "/af4a7426-c915-4fd8-a9a0-d1d0653890c7/c9470723-b410-4315-971f-b3c2471482a7"
-					(reference "#PWR?")
+					(reference "#PWR018")
 					(unit 1)
 				)
@@
 		(in_pos_files yes)
 		(dnp no)
-		(property "Reference" "#PWR?"
+		(property "Reference" "#PWR016"
 			(at 91.44 126.1872 0)
 			(hide yes)
@@
 			(project "Synapse_LPS"
 				(path "/af4a7426-c915-4fd8-a9a0-d1d0653890c7/c9470723-b410-4315-971f-b3c2471482a7"
-					(reference "#PWR?")
+					(reference "#PWR016")
 					(unit 1)
 				)
@@
 		(in_pos_files yes)
 		(dnp no)
-		(property "Reference" "#PWR?"
+		(property "Reference" "#PWR017"
 			(at 113.03 126.1872 0)
 			(hide yes)
@@
 			(project "Synapse_LPS"
 				(path "/af4a7426-c915-4fd8-a9a0-d1d0653890c7/c9470723-b410-4315-971f-b3c2471482a7"
-					(reference "#PWR?")
+					(reference "#PWR017")
 					(unit 1)
 				)
@@
 		(in_pos_files yes)
 		(dnp no)
-		(property "Reference" "#PWR?"
+		(property "Reference" "#PWR015"
 			(at 78.74 126.1872 0)
 			(hide yes)
@@
 			(project "Synapse_LPS"
 				(path "/af4a7426-c915-4fd8-a9a0-d1d0653890c7/c9470723-b410-4315-971f-b3c2471482a7"
-					(reference "#PWR?")
+					(reference "#PWR015")
 					(unit 1)
 				)
@@
 		(in_pos_files yes)
 		(dnp no)
-		(property "Reference" "RC2*"
+		(property "Reference" "RC2*1"
 			(at 98.806 89.6112 90)
 			(show_name no)
@@
 			(project "Synapse_LPS"
 				(path "/af4a7426-c915-4fd8-a9a0-d1d0653890c7/c9470723-b410-4315-971f-b3c2471482a7"
-					(reference "RC2*")
+					(reference "RC2*1")
 					(unit 1)
 				)
