File: PCBdesign/kicad/Synapse/Synapse_LPS.kicad_sch (KiCad schematic)
At the start: 12 parts, among them J1 SSW-102-01-G-S, J2 SSW-102-01-G-S, P1 TSW-102-07-G-S, P2 TSW-102-07-G-S, P3 TSW-102-07-G-S

Commit message: Annotate schematics (auto via kicad) and generate netlists.
Parts:
- renumbered R5* to R5*1, Ral* to Ral*1, Rex* to Rex*1
Changed lines of the file:
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@@
 		(in_pos_files yes)
 		(dnp no)
-		(property "Reference" "#PWR?"
+		(property "Reference" "#PWR023"
 			(at 154.94 60.1472 0)
 			(hide yes)
@@
 			(project "Synapse_LPS"
 				(path "/af4a7426-c915-4fd8-a9a0-d1d0653890c7"
-					(reference "#PWR?")
+					(reference "#PWR023")
 					(unit 1)
 				)
@@
 		(in_pos_files yes)
 		(dnp no)
-		(property "Reference" "R5*"
+		(property "Reference" "R5*1"
 			(at 211.836 131.0132 0)
 			(show_name no)
@@
 			(project "Synapse_LPS"
 				(path "/af4a7426-c915-4fd8-a9a0-d1d0653890c7"
-					(reference "R5*")
+					(reference "R5*1")
 					(unit 1)
 				)
@@
 		(in_pos_files yes)
 		(dnp no)
-		(property "Reference" "#PWR?"
+		(property "Reference" "#PWR024"
 			(at 157.48 52.5272 0)
 			(hide yes)
@@
 			(project "Synapse_LPS"
 				(path "/af4a7426-c915-4fd8-a9a0-d1d0653890c7"
-					(reference "#PWR?")
+					(reference "#PWR024")
 					(unit 1)
 				)
@@
 		(in_pos_files yes)
 		(dnp no)
-		(property "Reference" "#PWR?"
+		(property "Reference" "#PWR021"
 			(at 121.92 52.5272 0)
 			(hide yes)
@@
 			(project "Synapse_LPS"
 				(path "/af4a7426-c915-4fd8-a9a0-d1d0653890c7"
-					(reference "#PWR?")
+					(reference "#PWR021")
 					(unit 1)
 				)
@@
 		(in_pos_files yes)
 		(dnp no)
-		(property "Reference" "Ral*"
+		(property "Reference" "Ral*1"
 			(at 88.9 136.3472 90)
 			(show_name no)
@@
 			(project "Synapse_LPS"
 				(path "/af4a7426-c915-4fd8-a9a0-d1d0653890c7"
-					(reference "Ral*")
+					(reference "Ral*1")
 					(unit 1)
 				)
@@
 		(in_pos_files yes)
 		(dnp no)
-		(property "Reference" "#PWR?"
+		(property "Reference" "#PWR020"
 			(at 119.38 60.1472 0)
 			(hide yes)
@@
 			(project "Synapse_LPS"
 				(path "/af4a7426-c915-4fd8-a9a0-d1d0653890c7"
-					(reference "#PWR?")
+					(reference "#PWR020")
 					(unit 1)
 				)
@@
 		(in_pos_files yes)
 		(dnp no)
-		(property "Reference" "#PWR?"
+		(property "Reference" "#PWR026"
 			(at 175.26 52.5272 0)
 			(hide yes)
@@
 			(project "Synapse_LPS"
 				(path "/af4a7426-c915-4fd8-a9a0-d1d0653890c7"
-					(reference "#PWR?")
+					(reference "#PWR026")
 					(unit 1)
 				)
@@
 		(in_pos_files yes)
 		(dnp no)
-		(property "Reference" "#PWR?"
+		(property "Reference" "#PWR019"
 			(at 101.6 60.1472 0)
 			(hide yes)
@@
 			(project "Synapse_LPS"
 				(path "/af4a7426-c915-4fd8-a9a0-d1d0653890c7"
-					(reference "#PWR?")
+					(reference "#PWR019")
 					(unit 1)
 				)
@@
 		(in_pos_files yes)
 		(dnp no)
-		(property "Reference" "#PWR?"
+		(property "Reference" "#PWR025"
 			(at 172.72 60.1472 0)
 			(hide yes)
@@
 			(project "Synapse_LPS"
 				(path "/af4a7426-c915-4fd8-a9a0-d1d0653890c7"
-					(reference "#PWR?")
+					(reference "#PWR025")
 					(unit 1)
 				)
@@
 		(in_pos_files yes)
 		(dnp no)
-		(property "Reference" "#PWR?"
+		(property "Reference" "#PWR022"
 			(at 137.16 60.1472 0)
 			(hide yes)
@@
 			(project "Synapse_LPS"
 				(path "/af4a7426-c915-4fd8-a9a0-d1d0653890c7"
-					(reference "#PWR?")
+					(reference "#PWR022")
 					(unit 1)
 				)
@@
 		(in_pos_files yes)
 		(dnp no)
-		(property "Reference" "Rex*"
+		(property "Reference" "Rex*1"
 			(at 86.36 103.3272 90)
 			(show_name no)
@@
 			(project "Synapse_LPS"
 				(path "/af4a7426-c915-4fd8-a9a0-d1d0653890c7"
-					(reference "Rex*")
+					(reference "Rex*1")
 					(unit 1)
 				)
